Commit message: v3 before test shrinking

File: src/ar4_ros_driver/annin_ar4_moveit_config/urdf/fake_ar.urdf.xacro (robot description, xacro)
@@ -40,2 +40,43 @@
   />
 </robot>
+<?xml version="1.0"?>
+<robot xmlns:xacro="http://wiki.ros.org/xacro" name="$(arg ar_model)">
+  <xacro:include filename="$(find annin_ar4_description)/urdf/ar_macro.xacro"/>
+  <xacro:include filename="$(find annin_ar4_description)/urdf/ar_gripper_macro.xacro"/>
+  <xacro:include filename="$(find annin_ar4_description)/urdf/ar.ros2_control.xacro"/>
+  <xacro:include filename="$(find annin_ar4_description)/urdf/ar_gripper.ros2_control.xacro"/>
+  <!-- Load camera xacro -->
+  <xacro:include filename="$(find annin_ar4_description)/urdf/camera.xacro"/>
+  <!-- Call the macro and attach to base_link -->
+  <xacro:camera_link parent_link="base_link"/>
+  <xacro:arg name="tf_prefix" default="" />
+  <link name="world" />
+  <xacro:ar_robot
+    tf_prefix="$(arg tf_prefix)"
+    parent="world"
+    robot_parameters_file="$(find annin_ar4_description)/config/$(arg ar_model).yaml"
+  >
+    <origin xyz="0 0 0" rpy="0 0 0" />
+  </xacro:ar_robot>
+  <xacro:ar_gripper
+    tf_prefix="$(arg tf_prefix)"
+    parent="$(arg tf_prefix)ee_link"
+  />
+  <xacro:ar_ros2_control
+    ar_model="$(arg ar_model)"
+    plugin_name="mock_components/GenericSystem"
+    serial_port="/dev/ttyACM0"
+    calibrate="False"
+    robot_parameters_file="$(find annin_ar4_description)/config/$(arg ar_model).yaml"
+    joint_offset_parameters_file="$(find annin_ar4_driver)/config/joint_offsets/$(arg ar_model).yaml"
+    driver_parameters_file="$(find annin_ar4_driver)/config/driver.yaml"
+    tf_prefix="$(arg tf_prefix)"
+  />
+  <xacro:ar_gripper_ros2_control
+    name="ARGripperFakeSystem"
+    plugin_name="mock_components/GenericSystem"
+    serial_port="/dev/ttyUSB0"
+    driver_parameters_file="$(find annin_ar4_driver)/config/gripper_driver.yaml"
+    tf_prefix="$(arg tf_prefix)"
+  />
+</robot>
